Commit message: All axis is made positive 1, no neg in export parameters

File: Extras/URDF_Generation/scotty_description/urdf/scotty_description.urdf (robot description, URDF)
Before this commit: robot scotty_description, 13 links, 12 joints
Links:
- link knee_RR_link: mass 0.367874494498673 -> 0.367874494498672
Joints:
- joint abad_FL_joint: axis -0.999999999999999 0 0 -> 1 0 0; origin xyz=0.248499999209484 0.0649999995582956 0.0250000036169165 rpy=0 0 0 -> xyz=0.2485 0.065 0.025 rpy=0 0 0
- joint abad_FR_joint: axis -0.999999999999999 0 0 -> 1 0 0; origin xyz=0.248499999209484 -0.0650000004417044 0.0250000036169163 rpy=0 0 0 -> xyz=0.2485 -0.065 0.025 rpy=0 0 0
- joint abad_RL_joint: origin xyz=-0.248500000236906 0.0649999995582957 0.0249999944454496 rpy=0 0 0 -> xyz=-0.2485 0.065 0.025 rpy=0 0 0
- joint hip_FL_joint: axis 0 -1 0 -> 0 1 0; origin xyz=0.0649999999999999 0.0300000000000002 0 rpy=0 0 0 -> xyz=0.065 0.03 0 rpy=0 0 0
- joint hip_FR_joint: origin xyz=0.0649999999999999 -0.03 0 rpy=0 0 0 -> xyz=0.065 -0.03 0 rpy=0 0 0
- joint hip_RL_joint: axis 0 -1 0 -> 0 1 0; origin xyz=-0.065 0.0300000000000001 0 rpy=0 0 0 -> xyz=-0.065 0.03 0 rpy=0 0 0
- joint hip_RR_joint: origin xyz=-0.0650000000000002 -0.03 0 rpy=0 0 0 -> xyz=-0.065 -0.03 0 rpy=0 0 0
- joint knee_FL_joint: axis 0 -1 0 -> 0 1 0
- joint knee_FR_joint: origin xyz=0 -0.087404999999999 -0.3 rpy=0 0 0 -> xyz=0 -0.087405 -0.3 rpy=0 0 0
- joint knee_RL_joint: axis 0 -1 0 -> 0 1 0

Commit message: New URDF generated | foot added | inertia manually corrected

File: Extras/URDF_Generation/scotty_description/urdf/scotty_description.urdf (robot description, URDF)
Before this commit: robot scotty_description, 13 links, 12 joints
Links:
- added link foot_FL_link, mass 0.02; collision mesh filename=package://scotty_description/meshes/foot_FL_link.STL; visual mesh filename=package://scotty_description/meshes/foot_FL_link.STL
- added link foot_FR_link, mass 0.02; collision mesh filename=package://scotty_description/meshes/foot_FR_link.STL; visual mesh filename=package://scotty_description/meshes/foot_FR_link.STL
- added link foot_RL_link, mass 0.02; collision mesh filename=package://scotty_description/meshes/foot_RL_link.STL; visual mesh filename=package://scotty_description/meshes/foot_RL_link.STL
- added link foot_RR_link, mass 0.02; collision mesh filename=package://scotty_description/meshes/foot_RR_link.STL; visual mesh filename=package://scotty_description/meshes/foot_RR_link.STL
- link abad_FL_link: mass 0.415086538333225 -> 1.03
- link abad_FR_link: mass 0.415086541078643 -> 1.03
- link abad_RL_link: mass 0.415086538333242 -> 1.03
- link abad_RR_link: mass 0.415086541078617 -> 1.03
- link base_link: mass 3.85607896940888 -> 6.03
- link hip_FL_link: mass 1.05302815750899 -> 1.74
- link hip_FR_link: mass 1.05302815476358 -> 1.74
- link hip_RL_link: mass 1.05302815476357 -> 1.74
- link hip_RR_link: mass 1.05302815757229 -> 1.74
- link knee_FL_link: mass 0.367874494498672 -> 0.52
- link knee_FR_link: mass 0.367874494498672 -> 0.52
- link knee_RL_link: mass 0.367874494498672 -> 0.52
- link knee_RR_link: mass 0.367874494498672 -> 0.52
Joints:
- added joint foot_FL_joint: type fixed, parent knee_FL_link, child foot_FL_link, origin xyz=0.0175 0.004395 -0.3 rpy=0 0 0, axis 0 0 0
- added joint foot_FR_joint: type fixed, parent knee_FR_link, child foot_FR_link, origin xyz=0.0175 0.001605 -0.3 rpy=0 0 0, axis 0 0 0
- added joint foot_RL_joint: type fixed, parent knee_RL_link, child foot_RL_link, origin xyz=0.0175 0.004395 -0.3 rpy=0 0 0, axis 0 0 0
- added joint foot_RR_joint: type fixed, parent knee_RR_link, child foot_RR_link, origin xyz=0.0175 0.001605 -0.3 rpy=0 0 0, axis 0 0 0
