Commit message: new model | rviz is okay, gazebo not proper

File: Scotty_Champ/scotty_description/urdf/legs.xacro (robot description, xacro)
@@ -5,5 +5,12 @@
   <xacro:property name="lower_leg_to_foot_distance" value="0.32" />
   <!-- Front Right (FR) Foot -->
-  <link name="foot_FR_link" />
+  <link name="foot_FR_link">
+    <collision>
+      <origin xyz="0 0 -0.01" rpy="0 0 0" />
+      <geometry>
+        <box size="0.05 0.05 0.01"/>
+      </geometry>
+    </collision>
+  </link>
   <joint name="foot_FR_joint" type="fixed">
       <parent link="knee_FR_link" />
@@ -12,5 +19,12 @@
   </joint>
   <!-- Front Left (FL) Foot -->
-  <link name="foot_FL_link" />
+  <link name="foot_FL_link">
+    <collision>
+      <origin xyz="0 0 -0.01" rpy="0 0 0" />
+      <geometry>
+        <box size="0.05 0.05 0.01"/>
+      </geometry>
+    </collision>
+  </link>
   <joint name="foot_FL_joint" type="fixed">
       <parent link="knee_FL_link" />
@@ -19,5 +33,12 @@
   </joint>
   <!-- Rear Right (RR) Foot -->
-  <link name="foot_RR_link" />
+  <link name="foot_RR_link">
+    <collision>
+      <origin xyz="0 0 -0.01" rpy="0 0 0" />
+      <geometry>
+        <box size="0.05 0.05 0.01"/>
+      </geometry>
+    </collision>
+  </link>
   <joint name="foot_RR_joint" type="fixed">
       <parent link="knee_RR_link" />
@@ -26,5 +47,12 @@
   </joint>
   <!-- Rear Left (RL) Foot -->
-  <link name="foot_RL_link" />
+  <link name="foot_RL_link">
+    <collision>
+      <origin xyz="0 0 -0.01" rpy="0 0 0" />
+      <geometry>
+        <box size="0.05 0.05 0.01"/>
+      </geometry>
+    </collision>
+  </link>
   <joint name="foot_RL_joint" type="fixed">
       <parent link="knee_RL_link" />

File: Scotty_Champ/scotty_description/urdf/scotty.urdf (robot description, URDF)
Before this commit: robot scotty_robot, 19 links, 18 joints
Links:
- link abad_FL_link: mass 0.415086538333225 -> 1.03
- link abad_FR_link: mass 0.415086541078643 -> 1.03
- link abad_RL_link: mass 0.415086538333242 -> 1.03
- link abad_RR_link: mass 0.415086541078617 -> 1.03
- link base_link: mass 3.85607896940888 -> 6.03
- link foot_FL_link: mass None -> 0.02; geometry collision mesh filename=package://scotty_description/meshes/foot_FL_link.STL; visual mesh filename=package://scotty_description/meshes/foot_FL_link.STL
- link foot_FR_link: mass None -> 0.02; geometry collision mesh filename=package://scotty_description/meshes/foot_FR_link.STL; visual mesh filename=package://scotty_description/meshes/foot_FR_link.STL
- link foot_RL_link: mass None -> 0.02; geometry collision mesh filename=package://scotty_description/meshes/foot_RL_link.STL; visual mesh filename=package://scotty_description/meshes/foot_RL_link.STL
- link foot_RR_link: mass None -> 0.02; geometry collision mesh filename=package://scotty_description/meshes/foot_RR_link.STL; visual mesh filename=package://scotty_description/meshes/foot_RR_link.STL
- link hip_FL_link: mass 1.05302815750899 -> 1.74
- link hip_FR_link: mass 1.05302815476358 -> 1.74
- link hip_RL_link: mass 1.05302815476357 -> 1.74
- link hip_RR_link: mass 1.05302815757229 -> 1.74
- link knee_FL_link: mass 0.367874494498672 -> 0.52
- link knee_FR_link: mass 0.367874494498672 -> 0.52
- link knee_RL_link: mass 0.367874494498672 -> 0.52
- link knee_RR_link: mass 0.367874494498672 -> 0.52
Joints:
- joint foot_FL_joint: axis (none) -> 0 0 0; origin xyz=0 0 -0.32 rpy=0 0 0 -> xyz=0.0175 0.004395 -0.3 rpy=0 0 0
- joint foot_FR_joint: axis (none) -> 0 0 0; origin xyz=0 0 -0.32 rpy=0 0 0 -> xyz=0.0175 0.001605 -0.3 rpy=0 0 0
- joint foot_RL_joint: axis (none) -> 0 0 0; origin xyz=0 0 -0.32 rpy=0 0 0 -> xyz=0.0175 0.004395 -0.3 rpy=0 0 0
- joint foot_RR_joint: axis (none) -> 0 0 0; origin xyz=0 0 -0.32 rpy=0 0 0 -> xyz=0.0175 0.001605 -0.3 rpy=0 0 0

File: Scotty_Champ/scotty_description/urdf/scotty_description.urdf (robot description, URDF)
Before this commit: robot scotty_description, 13 links, 12 joints
Links:
- added link foot_FL_link, mass 0.02; collision mesh filename=package://scotty_description/meshes/foot_FL_link.STL; visual mesh filename=package://scotty_description/meshes/foot_FL_link.STL
- added link foot_FR_link, mass 0.02; collision mesh filename=package://scotty_description/meshes/foot_FR_link.STL; visual mesh filename=package://scotty_description/meshes/foot_FR_link.STL
- added link foot_RL_link, mass 0.02; collision mesh filename=package://scotty_description/meshes/foot_RL_link.STL; visual mesh filename=package://scotty_description/meshes/foot_RL_link.STL
- added link foot_RR_link, mass 0.02; collision mesh filename=package://scotty_description/meshes/foot_RR_link.STL; visual mesh filename=package://scotty_description/meshes/foot_RR_link.STL
- link abad_FL_link: mass 0.415086538333225 -> 1.03
- link abad_FR_link: mass 0.415086541078643 -> 1.03
- link abad_RL_link: mass 0.415086538333242 -> 1.03
- link abad_RR_link: mass 0.415086541078617 -> 1.03
- link base_link: mass 3.85607896940888 -> 6.03
- link hip_FL_link: mass 1.05302815750899 -> 1.74
- link hip_FR_link: mass 1.05302815476358 -> 1.74
- link hip_RL_link: mass 1.05302815476357 -> 1.74
- link hip_RR_link: mass 1.05302815757229 -> 1.74
- link knee_FL_link: mass 0.367874494498672 -> 0.52
- link knee_FR_link: mass 0.367874494498672 -> 0.52
- link knee_RL_link: mass 0.367874494498672 -> 0.52
- link knee_RR_link: mass 0.367874494498672 -> 0.52
Joints:
- added joint foot_FL_joint: type fixed, parent knee_FL_link, child foot_FL_link, origin xyz=0.0175 0.004395 -0.3 rpy=0 0 0, axis 0 0 0
- added joint foot_FR_joint: type fixed, parent knee_FR_link, child foot_FR_link, origin xyz=0.0175 0.001605 -0.3 rpy=0 0 0, axis 0 0 0
- added joint foot_RL_joint: type fixed, parent knee_RL_link, child foot_RL_link, origin xyz=0.0175 0.004395 -0.3 rpy=0 0 0, axis 0 0 0
- added joint foot_RR_joint: type fixed, parent knee_RR_link, child foot_RR_link, origin xyz=0.0175 0.001605 -0.3 rpy=0 0 0, axis 0 0 0

File: Scotty_Champ/scotty_description/urdf/scotty_final.urdf.xacro (robot description, xacro)
@@ -4,10 +4,8 @@
   <xacro:include filename="$(find scotty_description)/urdf/base.urdf.xacro" />
   <xacro:include filename="$(find scotty_description)/urdf/sensors.xacro" />
-  <!-- <xacro:include filename="$(find scotty_description)/urdf/transmissions.xacro" /> -->
-  <xacro:include filename="$(find scotty_description)/urdf/legs.xacro" />
+   <xacro:include filename="$(find scotty_description)/urdf/transmissions.xacro" />
   <!-- Invoke parts -->
   <xacro:base/>
   <xacro:sensors/>
-  <!-- <xacro:transmissions/> -->
-  <xacro:legs/>
+  <xacro:transmissions/>
 </robot>

File: Scotty_Champ/scotty_description/urdf/sensors.xacro (robot description, xacro)
@@ -29,4 +29,22 @@
         </plugin>
     </gazebo>
+    <!-- ros_control plugin -->
+    <gazebo>
+      <plugin name="p3d_base_controller" filename="libgazebo_ros_p3d.so">
+            <alwaysOn>true</alwaysOn>
+            <updateRate>10.0</updateRate>
+            <bodyName>base_link</bodyName>
+            <topicName>odom/ground_truth</topicName>
+            <gaussianNoise>0.01</gaussianNoise>
+            <frameName>world</frameName>
+            <xyzOffsets>0 0 0</xyzOffsets>
+            <rpyOffsets>0 0 0</rpyOffsets>
+        </plugin>
+    </gazebo>
+    <gazebo>
+        <plugin name="gazebo_ros_control" filename="libgazebo_ros_control.so">
+            <legacyModeNS>true</legacyModeNS>
+        </plugin>
+    </gazebo>
   </xacro:macro>
 </robot>
