Commit message: URDF corrected the trunk link | now base_link -> trunk -> abad

File: Scotty_Champ/scotty_description/urdf/scotty.urdf (robot description, URDF)
Before this commit: robot scotty_robot, 19 links, 18 joints
Joints:
- joint abad_FL_joint: parent base_link -> trunk
- joint abad_FR_joint: parent base_link -> trunk
- joint abad_RL_joint: parent base_link -> trunk
- joint abad_RR_joint: parent base_link -> trunk

File: Scotty_Champ/scotty_description/urdf/scotty_description.urdf (robot description, URDF)
Before this commit: robot scotty_description, 17 links, 16 joints
Joints:
- joint abad_FL_joint: parent base_link -> trunk
- joint abad_FR_joint: parent base_link -> trunk
- joint abad_RL_joint: parent base_link -> trunk
- joint abad_RR_joint: parent base_link -> trunk
