Commit message: Fixed xacro generation error | added name tag | successful generation of urdf

File: Scotty_Champ/scotty_description/urdf/base.urdf.xacro (robot description, xacro)
@@ -1,6 +1,7 @@
 <?xml version="1.0"?>
-<robot xmlns:xacro="http://ros.org/wiki/xacro" name="scotty_robot">
+<robot xmlns:xacro="http://ros.org/wiki/xacro">
+ <xacro:macro name="base">
   <!-- Include SolidWorks-generated URDF -->
-  <xacro:include filename="$(find scotty_description)/urdf/scotty_generated.urdf" />
+  <xacro:include filename="$(find scotty_description)/urdf/scotty_description.urdf" />
   <!-- Define base fixed joint -->
   <joint name="world_to_base" type="fixed">
@@ -9,3 +10,4 @@
     <origin xyz="0 0 0" rpy="0 0 0"/>
   </joint>
+ </xacro:macro>
 </robot>

File: Scotty_Champ/scotty_description/urdf/legs.xacro (robot description, xacro)
@@ -1,4 +1,5 @@
 <?xml version="1.0"?>
-<robot xmlns:xacro="http://ros.org/wiki/xacro" name="leg_description">
+<robot xmlns:xacro="http://ros.org/wiki/xacro">
+ <xacro:macro name="legs">
   <!-- Parameters -->
   <xacro:property name="lower_leg_to_foot_distance" value="0.32" />
@@ -31,3 +32,4 @@
       <origin xyz="0 0 -${lower_leg_to_foot_distance}" rpy="0 0 0" />
   </joint>
+ </xacro:macro>
 </robot>

File: Scotty_Champ/scotty_description/urdf/sensors.xacro (robot description, xacro)
@@ -1,4 +1,5 @@
 <?xml version="1.0"?>
 <robot xmlns:xacro="http://ros.org/wiki/xacro">
+  <xacro:macro name="sensors">
     <!-- IMU Link -->
     <link name="imu_link">
@@ -28,3 +29,4 @@
         </plugin>
     </gazebo>
+  </xacro:macro>
 </robot>

Commit message: URDF was improper | added world link | working

File: Scotty_Champ/scotty_description/urdf/base.urdf.xacro (robot description, xacro)
@@ -5,4 +5,5 @@
   <xacro:include filename="$(find scotty_description)/urdf/scotty_description.urdf" />
   <!-- Define base fixed joint -->
+  <link name="world" />
   <joint name="world_to_base" type="fixed">
     <parent link="world"/>

File: Scotty_Champ/scotty_description/urdf/scotty.urdf (robot description, URDF)
Before this commit: robot scotty_robot, 18 links, 18 joints
Links:
- added link world

Commit message: Updated the urdf | made trunk as parent link in solidworks | removed world link| added dynamics to joints

File: Scotty_Champ/scotty_description/urdf/base.urdf.xacro (robot description, xacro)
@@ -2,7 +2,21 @@
 <robot xmlns:xacro="http://ros.org/wiki/xacro">
  <xacro:macro name="base">
+  <link name="base_link">
+    <visual>
+      <origin rpy="0 0 0" xyz="0 0 0"/>
+      <geometry>
+        <box size="0.001 0.001 0.001"/>
+      </geometry>
+    </visual>
+  </link>
+  <joint name="floating_base_link" type="fixed">
+    <origin rpy="0 0 0" xyz="0 0 0"/>
+    <parent link="base_link"/>
+    <child link="trunk"/>
+  </joint>
   <!-- Include SolidWorks-generated URDF -->
   <xacro:include filename="$(find scotty_description)/urdf/scotty_description.urdf" />
-  <!-- Define base fixed joint -->
+<!--
+   Define base fixed joint
   <link name="world" />
   <joint name="world_to_base" type="fixed">
@@ -10,5 +24,5 @@
     <child link="base_link"/>
     <origin xyz="0 0 0" rpy="0 0 0"/>
-  </joint>
+  </joint> -->
  </xacro:macro>
 </robot>

File: Scotty_Champ/scotty_description/urdf/legs.xacro (robot description, xacro)
@@ -2,62 +2,40 @@
 <robot xmlns:xacro="http://ros.org/wiki/xacro">
  <xacro:macro name="legs">
-  <!-- Parameters -->
-  <xacro:property name="lower_leg_to_foot_distance" value="0.32" />
-  <!-- Front Right (FR) Foot -->
-  <link name="foot_FR_link">
-    <collision>
-      <origin xyz="0 0 -0.01" rpy="0 0 0" />
-      <geometry>
-        <box size="0.05 0.05 0.01"/>
-      </geometry>
-    </collision>
-  </link>
-  <joint name="foot_FR_joint" type="fixed">
-      <parent link="knee_FR_link" />
-      <child link="foot_FR_link" />
-      <origin xyz="0 0 -${lower_leg_to_foot_distance}" rpy="0 0 0" />
-  </joint>
-  <!-- Front Left (FL) Foot -->
-  <link name="foot_FL_link">
-    <collision>
-      <origin xyz="0 0 -0.01" rpy="0 0 0" />
-      <geometry>
-        <box size="0.05 0.05 0.01"/>
-      </geometry>
-    </collision>
-  </link>
-  <joint name="foot_FL_joint" type="fixed">
-      <parent link="knee_FL_link" />
-      <child link="foot_FL_link" />
-      <origin xyz="0 0 -${lower_leg_to_foot_distance}" rpy="0 0 0" />
-  </joint>
-  <!-- Rear Right (RR) Foot -->
-  <link name="foot_RR_link">
-    <collision>
-      <origin xyz="0 0 -0.01" rpy="0 0 0" />
-      <geometry>
-        <box size="0.05 0.05 0.01"/>
-      </geometry>
-    </collision>
-  </link>
-  <joint name="foot_RR_joint" type="fixed">
-      <parent link="knee_RR_link" />
-      <child link="foot_RR_link" />
-      <origin xyz="0 0 -${lower_leg_to_foot_distance}" rpy="0 0 0" />
-  </joint>
-  <!-- Rear Left (RL) Foot -->
-  <link name="foot_RL_link">
-    <collision>
-      <origin xyz="0 0 -0.01" rpy="0 0 0" />
-      <geometry>
-        <box size="0.05 0.05 0.01"/>
-      </geometry>
-    </collision>
-  </link>
-  <joint name="foot_RL_joint" type="fixed">
-      <parent link="knee_RL_link" />
-      <child link="foot_RL_link" />
-      <origin xyz="0 0 -${lower_leg_to_foot_distance}" rpy="0 0 0" />
-  </joint>
+<gazebo reference="foot_FR_link">
+    <kp>1000000.0</kp>
+    <kd>1.0</kd>
+    <mu1>0.8</mu1>
+    <mu2>0.8</mu2>
+    <maxVel>0.0</maxVel>
+    <minDepth>0.001</minDepth>
+    <material>Gazebo/FlatBlack</material>
+</gazebo>
+<gazebo reference="foot_FL_link">
+    <kp>1000000.0</kp>
+    <kd>1.0</kd>
+    <mu1>0.8</mu1>
+    <mu2>0.8</mu2>
+    <maxVel>0.0</maxVel>
+    <minDepth>0.001</minDepth>
+    <material>Gazebo/FlatBlack</material>
+</gazebo>
+<gazebo reference="foot_RR_link">
+    <kp>1000000.0</kp>
+    <kd>1.0</kd>
+    <mu1>0.8</mu1>
+    <mu2>0.8</mu2>
+    <maxVel>0.0</maxVel>
+    <minDepth>0.001</minDepth>
+    <material>Gazebo/FlatBlack</material>
+</gazebo>
+<gazebo reference="foot_RL_link">
+    <kp>1000000.0</kp>
+    <kd>1.0</kd>
+    <mu1>0.8</mu1>
+    <mu2>0.8</mu2>
+    <maxVel>0.0</maxVel>
+    <minDepth>0.001</minDepth>
+    <material>Gazebo/FlatBlack</material>
+</gazebo>
  </xacro:macro>
 </robot>

File: Scotty_Champ/scotty_description/urdf/scotty.urdf (robot description, URDF)
Before this commit: robot scotty_robot, 19 links, 18 joints
Links:
- removed link world
- added link trunk, mass 6.03; collision mesh filename=package://scotty_description/meshes/base_link.STL; visual mesh filename=package://scotty_description/meshes/base_link.STL
- link base_link: mass 6.03 -> None; geometry visual box size=0.001 0.001 0.001
Joints:
- removed joint world_to_base
- added joint floating_base_link: type fixed, parent base_link, child trunk, origin xyz=0 0 0 rpy=0 0 0
- joint abad_FL_joint: limit lower=-0.65 upper=0.65 effort=25 velocity=3 -> lower=-0.65 upper=0.65 effort=50 velocity=25
- joint abad_FR_joint: limit lower=-0.65 upper=0.65 effort=25 velocity=3 -> lower=-0.65 upper=0.65 effort=50 velocity=25
- joint abad_RL_joint: limit lower=-0.65 upper=0.65 effort=25 velocity=3 -> lower=-0.65 upper=0.65 effort=50 velocity=25
- joint abad_RR_joint: limit lower=-0.65 upper=0.65 effort=25 velocity=3 -> lower=-0.65 upper=0.65 effort=50 velocity=25
- joint hip_FL_joint: limit lower=-1.25 upper=1.8 effort=50 velocity=3 -> lower=-1.25 upper=1.8 effort=50 velocity=25
- joint hip_FR_joint: limit lower=-1.25 upper=1.8 effort=50 velocity=3 -> lower=-1.25 upper=1.8 effort=50 velocity=25
- joint hip_RL_joint: limit lower=-1.25 upper=1.8 effort=50 velocity=3 -> lower=-1.25 upper=1.8 effort=50 velocity=25
- joint hip_RR_joint: limit lower=-1.25 upper=1.8 effort=50 velocity=3 -> lower=-1.25 upper=1.8 effort=50 velocity=25
- joint knee_FL_joint: limit lower=-2.5 upper=0 effort=50 velocity=3 -> lower=-2.5 upper=0 effort=50 velocity=25
- joint knee_FR_joint: limit lower=-2.5 upper=0 effort=50 velocity=3 -> lower=-2.5 upper=0 effort=50 velocity=25
- joint knee_RL_joint: limit lower=-2.5 upper=0 effort=50 velocity=3 -> lower=-2.5 upper=0 effort=50 velocity=25
- joint knee_RR_joint: limit lower=-2.5 upper=0 effort=50 velocity=3 -> lower=-2.5 upper=0 effort=50 velocity=25

File: Scotty_Champ/scotty_description/urdf/scotty_description.urdf (robot description, URDF)
Before this commit: robot scotty_description, 17 links, 16 joints
Links:
- removed link base_link
- added link trunk, mass 6.03; collision mesh filename=package://scotty_description/meshes/base_link.STL; visual mesh filename=package://scotty_description/meshes/base_link.STL
Joints:
- joint abad_FL_joint: limit lower=-0.65 upper=0.65 effort=25 velocity=3 -> lower=-0.65 upper=0.65 effort=50 velocity=25
- joint abad_FR_joint: limit lower=-0.65 upper=0.65 effort=25 velocity=3 -> lower=-0.65 upper=0.65 effort=50 velocity=25
- joint abad_RL_joint: limit lower=-0.65 upper=0.65 effort=25 velocity=3 -> lower=-0.65 upper=0.65 effort=50 velocity=25
- joint abad_RR_joint: limit lower=-0.65 upper=0.65 effort=25 velocity=3 -> lower=-0.65 upper=0.65 effort=50 velocity=25
- joint hip_FL_joint: limit lower=-1.25 upper=1.8 effort=50 velocity=3 -> lower=-1.25 upper=1.8 effort=50 velocity=25
- joint hip_FR_joint: limit lower=-1.25 upper=1.8 effort=50 velocity=3 -> lower=-1.25 upper=1.8 effort=50 velocity=25
- joint hip_RL_joint: limit lower=-1.25 upper=1.8 effort=50 velocity=3 -> lower=-1.25 upper=1.8 effort=50 velocity=25
- joint hip_RR_joint: limit lower=-1.25 upper=1.8 effort=50 velocity=3 -> lower=-1.25 upper=1.8 effort=50 velocity=25
- joint knee_FL_joint: limit lower=-2.5 upper=0 effort=50 velocity=3 -> lower=-2.5 upper=0 effort=50 velocity=25
- joint knee_FR_joint: limit lower=-2.5 upper=0 effort=50 velocity=3 -> lower=-2.5 upper=0 effort=50 velocity=25
- joint knee_RL_joint: limit lower=-2.5 upper=0 effort=50 velocity=3 -> lower=-2.5 upper=0 effort=50 velocity=25
- joint knee_RR_joint: limit lower=-2.5 upper=0 effort=50 velocity=3 -> lower=-2.5 upper=0 effort=50 velocity=25

File: Scotty_Champ/scotty_description/urdf/scotty_final.urdf.xacro (robot description, xacro)
@@ -5,7 +5,9 @@
   <xacro:include filename="$(find scotty_description)/urdf/sensors.xacro" />
    <xacro:include filename="$(find scotty_description)/urdf/transmissions.xacro" />
+   <xacro:include filename="$(find scotty_description)/urdf/legs.xacro" />
   <!-- Invoke parts -->
   <xacro:base/>
   <xacro:sensors/>
   <xacro:transmissions/>
+  <xacro:legs/>
 </robot>

Commit message: RViz added for mode=hw | added back world frame | timeout for ros command in hw_interface

File: Scotty_Champ/scotty_description/urdf/base.urdf.xacro (robot description, xacro)
@@ -17,6 +17,5 @@
   <!-- Include SolidWorks-generated URDF -->
   <xacro:include filename="$(find scotty_description)/urdf/scotty_description.urdf" />
-<!--
-   Define base fixed joint
+   <!-- Define base fixed joint  -->
   <link name="world" />
   <joint name="world_to_base" type="fixed">
@@ -24,5 +23,5 @@
     <child link="base_link"/>
     <origin xyz="0 0 0" rpy="0 0 0"/>
-  </joint> -->
+  </joint>
  </xacro:macro>
 </robot>

File: Scotty_Champ/scotty_description/urdf/scotty.urdf (robot description, URDF)
Before this commit: robot scotty_robot, 19 links, 18 joints
Links:
- added link world
Joints:
- added joint world_to_base: type fixed, parent world, child base_link, origin xyz=0 0 0 rpy=0 0 0
